Commit message: camera restored

File: models/gupikModel/urdf/gupikModel.urdf (robot description, URDF)
Before this commit: robot gupikModel, 7 links, 6 joints
Links:
- added link mainCamera, mass 1e-5; visual box size=0.01 0.01 0.01
Joints:
- added joint mainCamera_joint: type fixed, parent base_link, child mainCamera, origin xyz=0 0 0 rpy=0 0 0, axis 0 1 0

Commit message: camera restored

File: models/gupikModel/urdf/gupikModel.urdf (robot description, URDF)
Before this commit: robot gupikModel, 8 links, 7 joints
Joints:
- joint mainCamera_joint: axis 0 1 0 -> 1 0 0; origin xyz=0 0 0 rpy=0 0 0 -> xyz=0.24 -0.021021 0.021021 rpy=0 0.129154365 0
